File: ESP01LEDDriver.kicad_sch (KiCad schematic)
At the start: 20 parts, among them CON1 POWERLJACK, J1 Conn_01x04, J2 Conn_02x04_Odd_Even, J3 Screw_Terminal_01x03, J4 USB_B, Q1 2N7002, SW1 RESETBUTTON, U1 AZ1117-3.3

Commit message: v2: added an FTDI IC for programming the ESP01 in place
This part is optional: if included on a built up board then the ESP01 can
be programmed without removing it from the board or using a USB UART
attached to the header pins.

Thanks to Phil Mehew (www.mehew.net) for this suggestion!
Parts:
- removed J4: USB_B, Connector_USB:USB_B_OST_USB-B1HSxx_Horizontal, symbol Connector:USB_B
- removed TP1: 3V3, TestPoint:TestPoint_Loop_D1.80mm_Drill1.0mm_Beaded, symbol Connector:TestPoint_Probe
- added C4: 10n, Capacitor_SMD:C_0805_2012Metric, symbol Device:C
- added C5, C6: 47p, Capacitor_SMD:C_0805_2012Metric, symbol Device:C
- added C7, C8: 4.7u, Capacitor_SMD:C_0805_2012Metric, symbol Device:C
- added D2, D3: UART_LED, LED_SMD:LED_1210_3225Metric, symbol Device:LED
- added FB1: Bead, Inductor_SMD:L_1206_3216Metric, symbol Device:FerriteBead
- added J5: USB_B, Connector_USB:USB_B_OST_USB-B1HSxx_Horizontal, symbol Connector:USB_B
- added R5, R6: 27, Resistor_SMD:R_0805_2012Metric, symbol Device:R
- added R7, R8: 1K, Resistor_SMD:R_0805_2012Metric, symbol Device:R
- added U2: FT231XS, Package_SO:SSOP-20_3.9x8.7mm_P0.635mm, symbol Interface_USB:FT231XS
- C1, C3: symbol Device:CP -> Device:C_Polarized
- C2: footprint Capacitor_SMD:C_1206_3216Metric -> Capacitor_SMD:C_0805_2012Metric
Connections:
- net RST is gone; now on net +3V3: J2.5 (Pin_5)
- net +3V3: now also C7.1, C8.1, D2.2 (A), D3.2 (A), U2.14 (~{RESET}), U2.3 (VCCIO)
- net +5V: now also FB1.1, U2.15 (VCC)
- net GND: now also C4.2, C5.2, C6.2, C7.2, C8.2, J5.4 (GND), J5.5 (Shield), U2.16 (GND), U2.6 (GND)
- net UART_RX: now also U2.20 (TXD)
- net UART_TX: now also U2.4 (RXD)
- new net: D2.1 (K), R7.1
- new net: R6.1, U2.11 (USBDP)
- new net: R5.1, U2.12 (USBDM)
- new net: C6.1, J5.3 (D+), R6.2
- new net: C5.1, J5.2 (D-), R5.2
- new net: D3.1 (K), R8.1
- new net RXLED: R8.2, U2.10 (CBUS2)
- new net TXLED: R7.2, U2.17 (CBUS1)
- new net VBUS: C4.1, FB1.2, J5.1 (VBUS)
- no-connect marks 2 -> 9
Other:
- note added: "CH_PD"
- note added: "RST"
- moved on the sheet: C1, C2, C3, H1, H2, H3, H4, J2, J3, Q1, R1, R2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
